File: keyboard-layout-pcb/keyboard-layout.kicad_pcb (KiCad board)
At the start: 2 copper layers, 50 x 196.7 mm, 33 parts, among them J1 Conn_01x06, J2 Conn_01x02, J3 Conn_01x02, Q1 IRLB871, U1 TSOP384xx, U2 TSMP58000, U3 RFM9xLoRa

Commit message: Updated MOSFET footprint and netlist
Parts:
- R1: value 620 -> 100
- R2, R3: value 620 -> 22
Connections:
- Q1 pad 3: +5V -> GND
Changed lines of the file:
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@@
     (zones 0)
     (modules 33)
-    (nets 44)
+    (nets 45)
   )
   (page A2 portrait)
@@
   (net 42 +5V)
   (net 43 3V)
+  (net 44 GND)
   (net_class Default "This is the default net class."
     (clearance 0.2)
@@
     (add_net +5V)
     (add_net 3V)
+    (add_net GND)
     (add_net "Net-(D1-Pad2)")
     (add_net "Net-(D1-Pad3)")
@@
     )
     (pad 3 thru_hole oval (at 5.08 0 180) (size 1.8 1.8) (drill 1) (layers *.Cu *.Mask)
-      (net 42 +5V))
+      (net 44 GND))
     (pad 2 thru_hole oval (at 2.54 0 180) (size 1.8 1.8) (drill 1) (layers *.Cu *.Mask)
       (net 15 "Net-(D2-Pad1)"))
@@
       (effects (font (size 1 1) (thickness 0.15)))
     )
-    (fp_text value 620 (at 6.35 2.86 90) (layer F.Fab)
+    (fp_text value 100 (at 6.35 2.86 90) (layer F.Fab)
       (effects (font (size 1 1) (thickness 0.15)))
     )
@@
       (effects (font (size 1 1) (thickness 0.15)))
     )
-    (fp_text value 620 (at 6.35 2.86 90) (layer F.Fab)
+    (fp_text value 22 (at 6.35 2.86 90) (layer F.Fab)
       (effects (font (size 1 1) (thickness 0.15)))
     )
@@
       (effects (font (size 1 1) (thickness 0.15)))
     )
-    (fp_text value 620 (at 6.35 2.86 90) (layer F.Fab)
-      (effects (font (size 1 1) (thickness 0.15)))
-    )
+    (fp_text value 22 (at 6.35 2.86 90) (layer F.Fab)
+      (effects (font (size 1 1) (thickness 0.15)))
+    )

Commit message: Edited a wiring issue, Added Remote Case, Added Key holder for laser engraving
Routing:
- net GND: track 0.00 -> 2.80 mm
- net +5V: track 244.6 -> 241.8 mm
Changed lines of the file:
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@@
     (35 F.Paste user)
     (36 B.SilkS user)
-    (37 F.SilkS user)
+    (37 F.SilkS user hide)
     (38 B.Mask user)
     (39 F.Mask user)
@@
   (segment (start 50.8 248.92) (end 49.72237 248.92) (width 0.25) (layer B.Cu) (net 40))
   (segment (start 50.8 246.38) (end 45.72 246.38) (width 0.25) (layer B.Cu) (net 41))
-  (segment (start 67.945 90.17) (end 67.945 88.265) (width 0.25) (layer B.Cu) (net 42) (status 20))
+  (segment (start 67.945 90.17) (end 67.945 88.265) (width 0.25) (layer B.Cu) (net 44) (status 20))
   (segment (start 85.725 254) (end 86.36 253.365) (width 0.25) (layer B.Cu) (net 42))
   (segment (start 71.12 254) (end 85.725 254) (width 0.25) (layer B.Cu) (net 42) (status 10))
   (segment (start 86.36 253.365) (end 86.36 92.075) (width 0.25) (layer B.Cu) (net 42))
   (segment (start 86.36 92.075) (end 85.09 90.805) (width 0.25) (layer B.Cu) (net 42))
-  (segment (start 85.09 90.805) (end 68.58 90.805) (width 0.25) (layer B.Cu) (net 42))
-  (segment (start 68.58 90.805) (end 67.945 90.17) (width 0.25) (layer B.Cu) (net 42))
-  (segment (start 67.945 81.915) (end 67.945 88.265) (width 0.25) (layer F.Cu) (net 42) (status 20))
+  (segment (start 68.58 90.805) (end 67.945 90.17) (width 0.25) (layer B.Cu) (net 44))
   (segment (start 67.945 81.915) (end 68.58 81.28) (width 0.25) (layer F.Cu) (net 42))
   (segment (start 68.58 81.28) (end 73.66 81.28) (width 0.25) (layer F.Cu) (net 42))
@@
   (segment (start 67.945 81.915) (end 67.945 74.93) (width 0.25) (layer F.Cu) (net 42))
   (segment (start 67.945 74.93) (end 66.675 73.66) (width 0.25) (layer F.Cu) (net 42))
+  (segment (start 85.09 90.805) (end 68.58 90.805) (width 0.25) (layer B.Cu) (net 42))
+  (segment (start 67.945 81.915) (end 67.945 88.265) (width 0.25) (layer F.Cu) (net 42) (status 20))
   (segment (start 57.785 86.36) (end 57.785 86.725) (width 0.25) (layer F.Cu) (net 43) (status 30))
   (segment (start 83.185 78.105) (end 76.835 78.105) (width 0.25) (layer B.Cu) (net 43))
